File: projects_flat/electrolama_oshcamp23_badge/version_current/working/working.sch (EAGLE design)
At the start: 2 parts

Commit message: fixed oshcamp pcb
Parts:
- removed J2: (no value), SparkFun-Connectors:CONN_10LOCK
- added ANT1: ANT3216LL00R2400A, ok-rf-dev:ANT-CERAMIC-YAGEO-ANT3216LL00R2400A
- added C1, C10, C18, C2, C3: 47u, ok-discretes-dev:CAP-1206
- added C11, C7: 8p, ok-discretes-dev:CAP-0402
- added C12, C14: 4u7, ok-discretes-dev:CAP-0402-NOTHERMALS
- added C13, C15, C16, C17, C20: 100n, ok-discretes-dev:CAP-0402-NOTHERMALS
- added C19, C4, C5, C6: 100n, ok-discretes-dev:CAP-0402
- added C8, C9: TBD, ok-discretes-dev:CAP-0402-NOTHERMALS
- added CON1: (no value), ok-connectors-dev:USBC_USB-C-12
- added CON2: STEMMA_I2C_QT, microbuilder:STEMMA_I2C_QT
- added D1: (no value), ok-discretes-dev:DIODE-SWITCHING-1N4148W
- added IC1: (no value), ok-chips-dev:INTERFACE-CH343G
- added IC2: LD1117-3.3, ok-chips-dev:POWER-LDO-LD1117-SOT223-4
- added IC3: WMCU-ESP8285H16, ok-chips-dev:WMCU-ESP8285H16
- added L1: TBD, ok-discretes-dev:INDUCTOR-0402
- added LED1: WS2812B5050, adafruit:WS2812B5050
- added MOD1: ESP-12S, ok-modules-dev:MODULE_ESP-12S
- added P1: Buzzer, ok-electromech-dev:PIEZO-MLT-8530
- added Q1, Q2, Q3: SS8050, ok-discretes-dev:NPN-MMBT5550LT1G
- added R1: 220, ok-discretes-dev:RES-0603
- added R10, R11, R4, R5, R6, R7, R8, R9: 12k 1%, ok-discretes-dev:RES-0402
- added R2, R3: 5k1, ok-discretes-dev:RES-0603
- added SJ1, SJ2, SJ3, SJ4: (no value), ok-mechanical-dev:SJ-SHORT
- added SW1, SW2, SW3, SW4, SW5, SW6, SW7: (no value), ok-electromech-dev:PUSHBUTTON-6X6MM
- added XT1: 26MHz, ok-xtal-osc-dev:XTAL-4P-2016
- J1: value (none) -> 61030621121; device SparkFun-Connectors:CONN_10LOCK -> Wurth_Connectors_WR-PHD:6103XX21121_61030621121; JLCASSY (none) -> C780054
Connections:
- removed net 3V3: J2.1, J2.2, J2.3, J2.4, J2.5
- new net ANT: C9.2, IC3.LNA, L1.2
- new net ANT': ANT1.FEED, C8.2, L1.1
- new net AUTORST_BOOT: J1.6, Q1.C, SJ4.1
- new net AUTORST_EN: J1.1, Q2.C, SJ1.2
- new net CH343_3V: C5.1, C6.1, IC1.V3, IC1.VIO
- new net DTR: IC1.DTR, Q1.E, R4.1
- new net EN: IC3.CHIP_EN, MOD1.EN, R7.2, SJ1.1
- new net IO0: IC3.GPIO0, MOD1.IO0, R8.2, SJ4.2, SW3.1
- new net IO13: IC3.MTCK, MOD1.IO13, R1.2
- new net IO1_TX: IC3.U0TXD, MOD1.TXD/IO1, SJ2.1
- new net IO2: IC3.GPIO2, MOD1.IO2, R9.2, SW4.1
- new net IO3_RX: IC3.U0RXD, MOD1.RXD/IO3, SJ3.1
- new net IO4: IC3.GPIO4, MOD1.IO4, SW2.1
- new net N$12: D1.A, P1.-, Q3.C
- new net N$13: Q2.B, R4.2
- new net N$16: CON1.CC1, R3.2
- new net N$17: CON1.CC2, R2.2
- new net N$23: Q3.B, R1.1
- new net N$5: Q1.B, R5.1
- new net N$6: IC3.RES12K, R6.1
- new net PC_RX: IC1.RXD, J1.3, SJ2.2
- new net PC_TX: IC1.TXD, J1.5, SJ3.2
- new net RST_C: C20.2, IC3.EXT_RSTB, R11.1
- new net RST_M: MOD1.RST
- new net RTS: IC1.RTS, Q2.E, R5.2
- new net USB_N: CON1.DN1, CON1.DN2, IC1.UD-
- new net USB_P: CON1.DP1, CON1.DP2, IC1.UD+
- new net VCC: C10.1, C12.2, C13.2, C14.2, C15.2, C16.2, C17.2, C18.1, C19.1, C2.1, C3.1, CON2G$1.V+, D1.C, IC2.TAB, IC2.VOUT, IC3.VDD3P3_1, IC3.VDD3P3_2, IC3.VDDA_1, IC3.VDDA_2, IC3.VDDD, IC3.VDDPST_1, IC3.VDDPST_2, J1.2, LED1.VDD, MOD1.VCC, P1.+, R11.2, R7.1, R8.1, R9.1, SW7.2
- new net VUSB: C1.1, C4.1, CON1.VBUS, IC1.VBUS, IC1.VDD5, IC2.VIN
- new net XTAL_IN: C7.2, IC3.XTAL_IN, XT1.1
- new net XTAL_OUT: C11.2, IC3.XTAL_OUT, XT1.3
- net GND: now also C1.2, C10.2, C11.1, C12.1, C13.1, C14.1, C15.1, C16.1, C17.1, C18.2, C19.2, C2.2, C20.1, C3.2, C4.2, C5.2, C6.2, C7.1, C8.1, C9.1, CON1.CHASSIS, CON1.GND, CON2G$1.GND, IC1.GND, IC2.GND, IC3.GND, J1.4, LED1.GND, MOD1.GND, Q3.E, R10.1, R2.1, R3.1, R6.2, SW1.2, SW2.2, SW3.2, SW4.2, SW5.2, SW6.2, XT1.2, XT1.4; no longer J1.10, J1.9, J2.10, J2.6, J2.7, J2.8, J2.9
- net IO12: now also CON2G$1.SCL, IC3.MTDI, MOD1.IO12, SW5.1; no longer J1.3, J1.4
- net IO14: now also CON2G$1.SDA, IC3.MTMS, MOD1.IO14, SW6.1; no longer J1.1, J1.2
- net IO15: now also IC3.MTDO, MOD1.IO15, R10.2, SW7.1; no longer J1.7, J1.8
- net IO5: now also IC3.GPIO5, LED1.DI, MOD1.IO5, SW1.1; no longer J1.5, J1.6
Other:
- note added: ""EXT_RSTB serves as the reset pin of ESP8266EX. This pin contains an internal pull-up resistor and is active low." "We recommend that you use CHIP_EN, instead of EXT_RSTB, to reset the chip." -ESP8266 HW Design Guidelines"
- note added: "** Resistors here do not need to be 1% but we are using the 12K 1% that we already have on the BOM to reduce the number of unique items we have on this board."
- note added: "5V -> 3.3V LDO"
- note added: "ANT1"
- note added: "Cut solder jumpers to turn this into an ESP-PROG compatible programmer (isolates the on-board ESP module and chip from CH343 UART)"
- note added: "DTR RTS -> Q1 Q2 EN BOOT 1 1 on on 1 1 0 0 off off 1 1 1 0 on off 0 1 0 1 off on 1 0"
- note added: "ESP Auto-Reset"
- note added: "ESP-12 Module"
- note added: "ESP8285H16 (ESP8266 + SPI FLASH)"
- note added: "I2C Port"
- note added: "IO15 is a bootstrap pin that needs to be pulled high at boot, hence the reason why it is different."
- note added: "Piezo Buzzer"
- note added: "Pushbuttons"
- note added: "RGB LED"
- note added: "This board is designed to be used as part of a solder paste workshop at OSHCamp 2023, also acting as a name badge, a generic sensor device using the qwiic/ stemma qt compatible I2C port and the Tasmota firmware and even a little piece of art, courtesy of OSHUG co-founder Paul Downey. You can also use it as a comically large USB-UART / ESP-Prog adapter for your other designs!! You'll notice both a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"
- note added: "U0RXD"
- note added: "U0TXD"
- note added: "UART/ESP-Prog Header"
- note added: "USB-C + USB-Serial"
- note added: "https://lab.electrolama.com/ob23 This open-source hardware design is licensed under the Solderpad Hardware License 2.0."
